File: PCB/PCB/PCB.kicad_sch (KiCad schematic)
At the start: 3 parts, among them U1 ESP32-C3-DEVKITM-1

Commit message: deleted unused pcb files
Parts:
- added J1: Conn_01x08_Socket, Connector_PinSocket_2.54mm:PinSocket_1x08_P2.54mm_Vertical, symbol Connector:Conn_01x08_Socket
Connections:
- net 5V: now also J1.8 (Pin_8)
- net GND: now also J1.1 (Pin_1)
Changed lines of the file:
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@@
+    )
+  )
+  (global_label "GND" (shape input) (at 116.84 80.01 0) (fields_autoplaced)
+    (effects (font (size 1.27 1.27)) (justify left))
+    (property "Intersheetrefs" "${INTERSHEET_REFS}" (at 123.6163 80.01 0)
+      (effects (font (size 1.27 1.27)) (justify left) hide)
     )
   )
@@
     (effects (font (size 1.27 1.27)) (justify left))
     (property "Intersheetrefs" "${INTERSHEET_REFS}" (at 130.81 102.4437 90)
+      (effects (font (size 1.27 1.27)) (justify left) hide)
+    )
+  )
+  (global_label "5V" (shape input) (at 116.84 62.23 0) (fields_autoplaced)
+    (effects (font (size 1.27 1.27)) (justify left))
+    (property "Intersheetrefs" "${INTERSHEET_REFS}" (at 122.0439 62.23 0)
       (effects (font (size 1.27 1.27)) (justify left) hide)
     )
@@
         )
       )
+    )
+  )
+  (symbol (lib_id "Connector:Conn_01x08_Socket") (at 111.76 72.39 180) (unit 1)
+    (in_bom yes) (on_board yes) (dnp no) (fields_autoplaced)
+    (property "Reference" "J1" (at 112.395 58.42 0)
+      (effects (font (size 1.27 1.27)))
+    )
+    (property "Value" "Conn_01x08_Socket" (at 112.395 60.96 0)
+      (effects (font (size 1.27 1.27)))
+    )
+    (property "Footprint" "Connector_PinSocket_2.54mm:PinSocket_1x08_P2.54mm_Vertical" (at 111.76 72.39 0)
+      (effects (font (size 1.27 1.27)) hide)
+    )
+    (property "Datasheet" "~" (at 111.76 72.39 0)
+      (effects (font (size 1.27 1.27)) hide)
+    )
+    (pin "1")
+    (pin "2")
+    (pin "3")
+    (pin "4")
+    (pin "5")
+    (pin "6")
+    (pin "7")
+    (pin "8")
+    (instances
+      (project "PCB"
+        (path "/a6f63534-8977-4ecc-ba64-740c7595bc23"
+          (reference "J1") (unit 1)
+        )
+      )
